Commit message: feat: make shelves solid so aisles constrain routing
The bottom shelf plate sat at z=0.30, spanning 0.26-0.34. The robot chassis tops
out at 0.194 and the wheels at 0.210, so nothing ever touched: robots drove
straight through shelf rows for free and the randomised layout had no effect on
how they moved through it. The corner posts do reach the floor, but they sit at
1 m spacing on the cell corners - exactly where a grid-centred robot is not.

Lowering the bottom plate to 0.18 makes it span 0.14-0.22, overlapping both the
chassis and the wheels by ~5 cm, so entering a shelf cell now generates real
contacts. Cartons stocked on that plate move down with it: add_cartons() reads
the same SHELF_HEIGHTS list, so the two cannot drift apart.

Chosen over blocking the move outright so the collision penalty does the work -
a wedged robot has to learn its way out rather than the env silently refusing.

Regenerate the URDFs after touching SHELF_HEIGHTS:
  .venv\Scripts\python.exe hivemind_env/assets/generate_shelves.py

File: hivemind_env/assets/shelf_1m.urdf (robot description, URDF)
Before this commit: robot shelf_1m, 34 links, 33 joints
Joints:
- joint carton_1_1_mount_joint: origin xyz=0.0000 0 0.3400 -> xyz=0.0000 0 0.2200
- joint shelf_1_joint: origin xyz=0 0 0.3 -> xyz=0 0 0.18

File: hivemind_env/assets/shelf_2m.urdf (robot description, URDF)
Before this commit: robot shelf_2m, 62 links, 61 joints
Joints:
- joint carton_1_1_mount_joint: origin xyz=-0.5000 0 0.3400 -> xyz=-0.5000 0 0.2200
- joint carton_1_2_mount_joint: origin xyz=0.5000 0 0.3400 -> xyz=0.5000 0 0.2200
- joint shelf_1_joint: origin xyz=0 0 0.3 -> xyz=0 0 0.18

File: hivemind_env/assets/shelf_3m.urdf (robot description, URDF)
Before this commit: robot shelf_3m, 90 links, 89 joints
Joints:
- joint carton_1_1_mount_joint: origin xyz=-1.0000 0 0.3400 -> xyz=-1.0000 0 0.2200
- joint carton_1_2_mount_joint: origin xyz=0.0000 0 0.3400 -> xyz=0.0000 0 0.2200
- joint carton_1_3_mount_joint: origin xyz=1.0000 0 0.3400 -> xyz=1.0000 0 0.2200
- joint shelf_1_joint: origin xyz=0 0 0.3 -> xyz=0 0 0.18

File: hivemind_env/assets/shelf_4m.urdf (robot description, URDF)
Before this commit: robot shelf_4m, 118 links, 117 joints
Joints:
- joint carton_1_1_mount_joint: origin xyz=-1.5000 0 0.3400 -> xyz=-1.5000 0 0.2200
- joint carton_1_2_mount_joint: origin xyz=-0.5000 0 0.3400 -> xyz=-0.5000 0 0.2200
- joint carton_1_3_mount_joint: origin xyz=0.5000 0 0.3400 -> xyz=0.5000 0 0.2200
- joint carton_1_4_mount_joint: origin xyz=1.5000 0 0.3400 -> xyz=1.5000 0 0.2200
- joint shelf_1_joint: origin xyz=0 0 0.3 -> xyz=0 0 0.18

File: hivemind_env/assets/shelf_5m.urdf (robot description, URDF)
Before this commit: robot shelf_5m, 146 links, 145 joints
Joints:
- joint carton_1_1_mount_joint: origin xyz=-2.0000 0 0.3400 -> xyz=-2.0000 0 0.2200
- joint carton_1_2_mount_joint: origin xyz=-1.0000 0 0.3400 -> xyz=-1.0000 0 0.2200
- joint carton_1_3_mount_joint: origin xyz=0.0000 0 0.3400 -> xyz=0.0000 0 0.2200
- joint carton_1_4_mount_joint: origin xyz=1.0000 0 0.3400 -> xyz=1.0000 0 0.2200
- joint carton_1_5_mount_joint: origin xyz=2.0000 0 0.3400 -> xyz=2.0000 0 0.2200
- joint shelf_1_joint: origin xyz=0 0 0.3 -> xyz=0 0 0.18

File: hivemind_env/assets/shelf_6m.urdf (robot description, URDF)
Before this commit: robot shelf_6m, 174 links, 173 joints
Joints:
- joint carton_1_1_mount_joint: origin xyz=-2.5000 0 0.3400 -> xyz=-2.5000 0 0.2200
- joint carton_1_2_mount_joint: origin xyz=-1.5000 0 0.3400 -> xyz=-1.5000 0 0.2200
- joint carton_1_3_mount_joint: origin xyz=-0.5000 0 0.3400 -> xyz=-0.5000 0 0.2200
- joint carton_1_4_mount_joint: origin xyz=0.5000 0 0.3400 -> xyz=0.5000 0 0.2200
- joint carton_1_5_mount_joint: origin xyz=1.5000 0 0.3400 -> xyz=1.5000 0 0.2200
- joint carton_1_6_mount_joint: origin xyz=2.5000 0 0.3400 -> xyz=2.5000 0 0.2200
- joint shelf_1_joint: origin xyz=0 0 0.3 -> xyz=0 0 0.18

File: hivemind_env/assets/shelf_7m.urdf (robot description, URDF)
Before this commit: robot shelf_7m, 202 links, 201 joints
Joints:
- joint carton_1_1_mount_joint: origin xyz=-3.0000 0 0.3400 -> xyz=-3.0000 0 0.2200
- joint carton_1_2_mount_joint: origin xyz=-2.0000 0 0.3400 -> xyz=-2.0000 0 0.2200
- joint carton_1_3_mount_joint: origin xyz=-1.0000 0 0.3400 -> xyz=-1.0000 0 0.2200
- joint carton_1_4_mount_joint: origin xyz=0.0000 0 0.3400 -> xyz=0.0000 0 0.2200
- joint carton_1_5_mount_joint: origin xyz=1.0000 0 0.3400 -> xyz=1.0000 0 0.2200
- joint carton_1_6_mount_joint: origin xyz=2.0000 0 0.3400 -> xyz=2.0000 0 0.2200
- joint carton_1_7_mount_joint: origin xyz=3.0000 0 0.3400 -> xyz=3.0000 0 0.2200
- joint shelf_1_joint: origin xyz=0 0 0.3 -> xyz=0 0 0.18
