Commit message: base

File: hivemind_env/assets/diff_drive_bot.urdf (robot description, URDF)
Before this commit: robot diff_drive_bot, 12 links, 11 joints
Links:
- link gripper_palm_link: geometry visual box size=0.024 0.52 0.024
- link left_finger_link: geometry visual box size=0.12 0.016 0.028
- link lidar_post_link: geometry visual cylinder length=0.30 radius=0.012
- link right_finger_link: geometry visual box size=0.12 0.016 0.028
Joints:
- joint left_finger_joint: origin xyz=0.0 0.06 0.0 rpy=0 0 0 -> xyz=0.0 0.26 0.0 rpy=0 0 0
- joint lidar_joint: limit lower=0.0 upper=0.14 effort=10.0 velocity=1.0 -> lower=0.0 upper=0.50 effort=10.0 velocity=1.0
- joint right_finger_joint: origin xyz=0.0 -0.06 0.0 rpy=0 0 0 -> xyz=0.0 -0.26 0.0 rpy=0 0 0

Commit message: fixed env

File: hivemind_env/assets/diff_drive_bot.urdf (robot description, URDF)
Before this commit: robot diff_drive_bot, 12 links, 11 joints
Links:
- added link arm_lift_link, mass 0.05
- link lidar_post_link: geometry visual cylinder length=0.48 radius=0.012
Joints:
- added joint arm_lift_joint: type prismatic, parent lidar_post_link, child arm_lift_link, origin xyz=0.0 0.0 0.10 rpy=0 0 0, axis 0 0 1, limit lower=0.0 upper=0.38 effort=10.0 velocity=1.0
- joint arm_yaw_joint: origin xyz=0.0 0.0 0.14 rpy=0 0 0 -> xyz=0.0 0.0 0.0 rpy=0 0 0; parent base_link -> arm_lift_link
- joint lidar_joint: axis 0 0 1 -> (none); limit lower=0.0 upper=0.50 effort=10.0 velocity=1.0 -> (none); type prismatic -> fixed
